File: Laptop mods/nvme_ae_to_m/nvme_ae_to_m.kicad_sch (KiCad schematic)
At the start: 9 parts

Commit message: Initial commit with new footprint and placement
Parts:
- removed J1: (no value), symbol Connector_Generic:Conn_01x04
- added J1: USB, nvme_ae_to_m:BL-R8812AF1, symbol Connector:Conn_01x12_Pin
- C1, C2: value (none) -> 10uF; footprint (none) -> Capacitor_SMD:C_1206_3216Metric_Pad1.33x1.80mm_HandSolder
- R1, R2, R3, R4: value (none) -> 0R; footprint (none) -> Resistor_SMD:R_0603_1608Metric_Pad0.98x0.95mm_HandSolder
- U1: value (none) -> NGFF_M; footprint (none) -> nvme_ae_to_m:Conn_TE-M.2-0.5-67P-doublesided_TypeM
- U2: value (none) -> NGFF_AE; footprint (none) -> nvme_ae_to_m:NGFF_A+E
Connections:
- net +3V3: now also J1.2 (Pin_2)
- net D+: now also J1.4 (Pin_4)
- net D-: now also J1.3 (Pin_3)
- net GND: now also J1.10 (Pin_10), J1.12 (Pin_12), J1.5 (Pin_5), J1.7 (Pin_7), J1.9 (Pin_9)
