File: Laptop mods/nvme_ae_to_m/nvme_ae_to_m.kicad_pcb (KiCad board)
At the start: 2 copper layers, 22 x 26 mm, 9 parts, among them J1 USB, U1 NGFF_M, U2 NGFF_AE

Commit message: Extend length, fill zones.
Parts:
- removed C1, C2: 10uF, Capacitor_SMD:C_1206_3216Metric_Pad1.33x1.80mm_HandSolder
- moved J1 15.0 mm to (137.1, 137.0)
Routing:
- net (no net): track 0.00 -> 65.6 mm
- net D-: track 4.84 -> 3.65 mm, vias 1 -> 0
- net D+: vias 1 -> 0
Other:
- board size 22 x 26 mm -> 22 x 58.9 mm
